File: KiCad/ardAudioCenter-ams1117/ardAudioCenter-ams1117.kicad_sch (KiCad schematic)
At the start: 31 parts, among them J1 AudioPlug3, J2 Audio out, J3 LCD, J4 FM In, J5 Line In, U1 2-pole_power_in_screw_terminal, U10 MCP41010, U11 VolR, U12 FM Radio, U2 Rotary encoder 2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

Commit message: kicad
Parts:
- U6: value JDY-62_Bluetooth_Module -> JDY-62 Bluetooth
Other:
- note added: "black"
- note added: "green"
- note added: "grey"
- note added: "orange"
- note added: "red"
- note added: "white"
- note added: "yellow"
- moved on the sheet: J3, J4, J5, U11, U2, U4, U5, U6
