File: KiCad/ardAudioCenter-ams1117-autorouted/ardAudioCenter-ams1117-autorouted.kicad_pcb (KiCad board)
At the start: 2 copper layers, 99.7 x 69.2 mm, 30 parts, among them J2 Audio out, J3 LCD, J4 FM In, J5 Line In, U1 2-pole_power_in_screw_terminal, U10 MCP41010, U11 VolR, U12 FM Radio TEA5767, U2 Rotary encoder 2, U3 AMS1117-5.0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

Commit message: kicad
Parts:
- U11, U8: footprint My_Misc:JST_XH_B3B-XH-A_1x03_P2.50mm_Vertical large -> My_Headers:3-pin JST Potentiometer

Commit message: new 3D
Parts:
- U1: value 2-pole_power_in_screw_terminal -> Power In
- U10, U7: footprint My_Misc:DIP-8_W7.62mm_large -> My_Misc:DIP-8_W7.62mm_Socket_w_dip_packet_LongPads
- U9: footprint My_Misc:DIP-16_W7.62mm_larger -> My_Misc:DIP-16_W7.62mm_LongPads w socket
