File: KiCad/ardAudioCenter-ams1117-autorouted/ardAudioCenter-ams1117-autorouted.kicad_sch (KiCad schematic)
At the start: 31 parts, among them J1 AudioPlug3, J2 Audio out, J3 LCD, J4 FM In, J5 Line In, U1 2-pole_power_in_screw_terminal, U10 MCP41010, U11 VolR, U12 FM Radio, U2 Rotary encoder 2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

Commit message: 2-layer PCB
Parts:
- U12: value FM Radio -> FM Radio TEA5767
Other:
- moved on the sheet: U12

Commit message: kicad
Parts:
- U11, U8: footprint My_Misc:JST_XH_B3B-XH-A_1x03_P2.50mm_Vertical large -> My_Headers:3-pin JST Potentiometer
Changed lines of the file:
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@@
       (effects (font (size 1.27 1.27)) (justify left))
     )
-    (property "Footprint" "My_Misc:JST_XH_B3B-XH-A_1x03_P2.50mm_Vertical large" (id 2) (at 248.285 133.35 0)
+    (property "Footprint" "My_Headers:3-pin JST Potentiometer" (id 2) (at 248.285 133.35 0)
       (effects (font (size 1.27 1.27)) hide)
     )
@@
       (effects (font (size 1.27 1.27)) (justify left))
     )
-    (property "Footprint" "My_Misc:JST_XH_B3B-XH-A_1x03_P2.50mm_Vertical large" (id 2) (at 193.675 133.35 0)
+    (property "Footprint" "My_Headers:3-pin JST Potentiometer" (id 2) (at 193.675 133.35 0)
       (effects (font (size 1.27 1.27)) hide)
     )
@@
     )
     (path "/00000000-0000-0000-0000-00005ee9ceae"
-      (reference "U8") (unit 1) (value "VolL") (footprint "My_Misc:JST_XH_B3B-XH-A_1x03_P2.50mm_Vertical large")
+      (reference "U8") (unit 1) (value "VolL") (footprint "My_Headers:3-pin JST Potentiometer")
     )
     (path "/00000000-0000-0000-0000-00005ecc0ed1"
@@
     )
     (path "/00000000-0000-0000-0000-00005ee9c6fe"
-      (reference "U11") (unit 1) (value "VolR") (footprint "My_Misc:JST_XH_B3B-XH-A_1x03_P2.50mm_Vertical large")
+      (reference "U11") (unit 1) (value "VolR") (footprint "My_Headers:3-pin JST Potentiometer")
     )
     (path "/00000000-0000-0000-0000-00005ed4f406"

Commit message: minor changes
Parts:
- J1: value AudioPlug3 -> FM Audio Plug
- U1: value 2-pole_power_in_screw_terminal -> Power In
Changed lines of the file:
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@@
     (in_bom yes) (on_board yes)
     (property "Reference" "U5" (id 0) (at 71.755 66.4718 0))
-    (property "Value" "Rotary encoder 1" (id 1) (at 71.755 64.77 0)
-      (effects (font (size 1.27 1.27)) hide)
-    )
+    (property "Value" "Rotary encoder 1" (id 1) (at 71.755 64.77 0))
     (property "Footprint" "My_Headers:5-pin JST Rotary Encoder" (id 2) (at 73.025 67.31 0)
       (effects (font (size 1.27 1.27)) hide)
@@
     (in_bom yes) (on_board yes)
     (property "Reference" "U2" (id 0) (at 32.385 116.0018 0))
-    (property "Value" "Rotary encoder 2" (id 1) (at 32.385 114.3 0)
-      (effects (font (size 1.27 1.27)) hide)
-    )
+    (property "Value" "Rotary encoder 2" (id 1) (at 32.385 114.3 0))
     (property "Footprint" "My_Headers:5-pin JST Rotary Encoder" (id 2) (at 33.655 116.84 0)
       (effects (font (size 1.27 1.27)) hide)
@@
     (in_bom yes) (on_board yes)
     (property "Reference" "J1" (id 0) (at 101.7778 16.0782 0))
-    (property "Value" "AudioPlug3" (id 1) (at 101.7778 18.3896 0))
+    (property "Value" "FM Audio Plug" (id 1) (at 101.7778 18.3896 0))
     (property "Footprint" "" (id 2) (at 102.87 26.67 0)
       (effects (font (size 1.27 1.27)) hide)
@@
     (in_bom yes) (on_board yes)
     (property "Reference" "U1" (id 0) (at 29.718 33.655 0))
-    (property "Value" "2-pole_power_in_screw_terminal" (id 1) (at 29.718 35.9664 0))
+    (property "Value" "Power In" (id 1) (at 29.718 35.9664 0))
     (property "Footprint" "My_Parts:2-pole_power_in_screw_terminal" (id 2) (at 29.845 36.195 0)
       (effects (font (size 1.27 1.27)) hide)
@@
     )
     (path "/00000000-0000-0000-0000-00005edb2ee3"
-      (reference "J1") (unit 1) (value "AudioPlug3") (footprint "")
+      (reference "J1") (unit 1) (value "FM Audio Plug") (footprint "")
     )
     (path "/829b6792-e231-4abe-acac-47904b6d7e0b"
@@
     )
     (path "/00000000-0000-0000-0000-00005ee57baf"
-      (reference "U1") (unit 1) (value "2-pole_power_in_screw_terminal") (footprint "My_Parts:2-pole_power_in_screw_terminal")
+      (reference "U1") (unit 1) (value "Power In") (footprint "My_Parts:2-pole_power_in_screw_terminal")
     )
     (path "/00000000-0000-0000-0000-00005ecc58c0"

Commit message: new 3D
Parts:
- U10, U7: footprint My_Misc:DIP-8_W7.62mm_large -> My_Misc:DIP-8_W7.62mm_Socket_w_dip_packet_LongPads
- U9: footprint My_Misc:DIP-16_W7.62mm_larger -> My_Misc:DIP-16_W7.62mm_LongPads w socket
Changed lines of the file:
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@@
     (property "Reference" "U9" (id 0) (at 200.66 30.9626 0))
     (property "Value" "CD4052B" (id 1) (at 200.66 33.274 0))
-    (property "Footprint" "My_Misc:DIP-16_W7.62mm_larger" (id 2) (at 204.47 72.39 0)
+    (property "Footprint" "My_Misc:DIP-16_W7.62mm_LongPads w socket" (id 2) (at 204.47 72.39 0)
       (effects (font (size 1.27 1.27)) (justify left) hide)
     )
@@
     (property "Reference" "U7" (id 0) (at 175.26 123.6726 0))
     (property "Value" "MCP41010" (id 1) (at 175.26 125.984 0))
-    (property "Footprint" "My_Misc:DIP-8_W7.62mm_large" (id 2) (at 175.26 138.43 0)
+    (property "Footprint" "My_Misc:DIP-8_W7.62mm_Socket_w_dip_packet_LongPads" (id 2) (at 175.26 138.43 0)
       (effects (font (size 1.27 1.27)) hide)
     )
@@
     (property "Reference" "U10" (id 0) (at 229.87 123.6726 0))
     (property "Value" "MCP41010" (id 1) (at 229.87 125.984 0))
-    (property "Footprint" "My_Misc:DIP-8_W7.62mm_large" (id 2) (at 229.87 138.43 0)
+    (property "Footprint" "My_Misc:DIP-8_W7.62mm_Socket_w_dip_packet_LongPads" (id 2) (at 229.87 138.43 0)
       (effects (font (size 1.27 1.27)) hide)
     )
@@
     )
     (path "/00000000-0000-0000-0000-00005ecc220d"
-      (reference "U7") (unit 1) (value "MCP41010") (footprint "My_Misc:DIP-8_W7.62mm_large")
+      (reference "U7") (unit 1) (value "MCP41010") (footprint "My_Misc:DIP-8_W7.62mm_Socket_w_dip_packet_LongPads")
     )
     (path "/00000000-0000-0000-0000-00005ee9ceae"
@@
     )
     (path "/00000000-0000-0000-0000-00005ecc0ed1"
-      (reference "U9") (unit 1) (value "CD4052B") (footprint "My_Misc:DIP-16_W7.62mm_larger")
+      (reference "U9") (unit 1) (value "CD4052B") (footprint "My_Misc:DIP-16_W7.62mm_LongPads w socket")
     )
     (path "/00000000-0000-0000-0000-00005ecc2a42"
-      (reference "U10") (unit 1) (value "MCP41010") (footprint "My_Misc:DIP-8_W7.62mm_large")
+      (reference "U10") (unit 1) (value "MCP41010") (footprint "My_Misc:DIP-8_W7.62mm_Socket_w_dip_packet_LongPads")
     )
     (path "/00000000-0000-0000-0000-00005ee9c6fe"
