File: KiCad/DualTDA2005Amplifier/DualTDA2005Amplifier.kicad_sch (KiCad schematic)
At the start: 40 parts, among them U1 TDA2005, U2 TDA2005

Commit message: Dual amplifier
Parts:
- added H1, H2, H3, H4: MountingHole, MountingHole:MountingHole_3.2mm_M3, symbol Mechanical:MountingHole
- added HS1: Heatsink, My_Heatsinks:Heatsink SK81 100x37.5x15, symbol Mechanical:Heatsink
- added U3: Speakers out, My_Parts:4-pole_screw_terminal_RL_output, symbol My_Parts:4-pole_RL-output_screw_terminal
- added U4: Power in, My_Parts:2-pole_power_in_screw_terminal, symbol My_Parts:2-pole_power_in_screw_terminal
- added U5: Audio in, My_Headers:3-pin JST Audio, symbol My_Parts:3-pole_RL-input_screw_terminal
Connections:
- net GND: now also U4.2 (-), U5.3 (GND)
- net Left In: now also U5.2 (Lin)
- net Left Out +: now also U3.3 (Lout+)
- net Left Out -: now also U3.4 (Lout-)
- net Right In: now also U5.1 (Rin)
- net Right Out +: now also U3.1 (Rout+)
- net Right Out -: now also U3.2 (Rout-)
- net VCC: now also U4.1 (+)
