File: KiCad/DualTDA2005Amplifier/DualTDA2005Amplifier.kicad_pcb (KiCad board)
At the start: 2 copper layers, 40 parts, among them U1 TDA2005, U2 TDA2005

Commit message: Dual amplifier
Parts:
- added H1: MountingHole, MountingHole:MountingHole_3.2mm_M3, F.Cu at (118.1, 98.4)
- added H2: MountingHole, MountingHole:MountingHole_3.2mm_M3, F.Cu at (118.1, 52.7)
- added H3: MountingHole, MountingHole:MountingHole_3.2mm_M3, F.Cu at (210.2, 98.4)
- added H4: MountingHole, MountingHole:MountingHole_3.2mm_M3, F.Cu at (210.2, 52.7)
- added HS1: Heatsink, My_Heatsinks:Heatsink SK81 100x37.5x15, F.Cu at (114.6, 48.7)
- added U3: Speakers out, My_Parts:4-pole_screw_terminal_RL_output, F.Cu at (165.9, 96.3)
- added U4: Power in, My_Parts:2-pole_power_in_screw_terminal, F.Cu at (148.5, 96.3)
- added U5: Audio in, My_Headers:3-pin JST Audio, F.Cu at (140.3, 96.5)
- moved U1 161.4 mm to (132.9, 58.4)
- moved C12 157.3 mm to (149.9, 70.5), turned to -90 degrees
- moved C9 151.8 mm to (154.4, 63.5)
- moved R6 147.6 mm to (161.9, 63.5), turned to -90 degrees
- moved C10 146.3 mm to (141.3, 74.3)
- moved C3 141.3 mm to (156.9, 88.9)
- moved RV1 140.6 mm to (128.2, 91.8), turned to 180 degrees
- moved R4 136.4 mm to (146.1, 67.9), turned to 180 degrees
- moved C2 129.8 mm to (132.7, 80.0), turned to -90 degrees
- moved C7 129.6 mm to (134.6, 73.7), turned to -90 degrees
- moved R5 129.2 mm to (155.6, 72.4), turned to -90 degrees
- moved C8 125.8 mm to (154.9, 53.3)
- moved C1 125.7 mm to (149.2, 84.5), turned to 180 degrees
- moved C5 118.5 mm to (126.4, 52.4), turned to -90 degrees
- moved C11 114.9 mm to (161.9, 78.1), turned to -90 degrees
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Connections:
- net /Left Out + renamed Left Out +
- net /Left Out - renamed Left Out -
- net /Right Out + renamed Right Out +
- net /Right Out - renamed Right Out -
- RV1 pad 1: /Left In -> Left In
- RV2 pad 1: /Right In -> Right In
Routing:
- net GND: track 125.9 -> 288.4 mm
- net VCC: track 39.3 -> 148.2 mm
- net Left Out +: track 0.00 -> 79.8 mm
- net Left Out -: track 0.00 -> 76.1 mm
- net Right In: track 0.00 -> 69.5 mm
- net Right Out -: track 36.5 -> 99.6 mm
- net Net-(C6-Pad1): track 0.00 -> 37.7 mm
- net Net-(C2-Pad2): track 0.00 -> 23.6 mm
- net Right Out +: track 66.0 -> 83.4 mm
- net Net-(C7-Pad1): track 0.00 -> 17.3 mm
- net Net-(C20-Pad1): track 5.08 -> 20.8 mm
- net Net-(C14-Pad2): track 16.1 -> 31.6 mm
- net Net-(C9-Pad1): track 0.00 -> 14.2 mm
- net Net-(C12-Pad1): track 0.00 -> 13.6 mm
- net Net-(C5-Pad1): track 0.00 -> 12.8 mm
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- added copper zone on B.Cu, net GND
- added copper zone on F.Cu, net GND
Other:
- board outline added: 98.4 x 67.9 mm
- board text added: "DualTDA2005Amplifier Design: Jon Sagebrand github.com/jonsag/ardAudioCenter"
- board text added: "Left"
- board text added: "Right"

Commit message: PCBs
Changed lines of the file:
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@@
       (outputformat 1)
       (mirror false)
-      (drillshape 1)
+      (drillshape 0)
       (scaleselection 1)
-      (outputdirectory "")
+      (outputdirectory "Gerber")
     )
   )
@@
     (fp_line (start 7.45 -2.35) (end -2.45 -2.35) (layer "F.Fab") (width 0.1))
     (fp_line (start -2.45 -2.35) (end -2.45 3.4) (layer "F.Fab") (width 0.1))
-    (pad "1" thru_hole roundrect (at 0 0 180) (size 1.7 2.032) (drill 0.95) (layers *.Cu *.Mask) (roundrect_rratio 0.147059)
+    (pad "1" thru_hole roundrect (at 0 0 180) (size 1.7 2.032) (drill 0.95) (layers *.Cu *.Mask) (roundrect_rratio 0.1470588235)
       (net 34 "Right In") (pinfunction "Rin") (pintype "input"))
     (pad "2" thru_hole oval (at 2.5 0 180) (size 1.7 2.032) (drill 0.95) (layers *.Cu *.Mask)
@@
     (fp_line (start 0 -1.35) (end 0.625 -2.35) (layer "F.Fab") (width 0.1))
     (fp_line (start -2.45 3.4) (end 7.45 3.4) (layer "F.Fab") (width 0.1))
-    (pad "1" thru_hole roundrect (at 0 0 180) (size 1.7 2.032) (drill 0.95) (layers *.Cu *.Mask) (roundrect_rratio 0.147059)
+    (pad "1" thru_hole roundrect (at 0 0 180) (size 1.7 2.032) (drill 0.95) (layers *.Cu *.Mask) (roundrect_rratio 0.1470588235)
       (net 34 "Right In") (pinfunction "1") (pintype "passive"))
     (pad "2" thru_hole oval (at 2.5 0 180) (size 1.7 2.032) (drill 0.95) (layers *.Cu *.Mask)
@@
     (fp_line (start -2.45 -2.35) (end -2.45 3.4) (layer "F.Fab") (width 0.1))
     (fp_line (start 7.45 3.4) (end 7.45 -2.35) (layer "F.Fab") (width 0.1))
-    (pad "1" thru_hole roundrect (at 0 0 180) (size 1.7 2.032) (drill 0.95) (layers *.Cu *.Mask) (roundrect_rratio 0.147059)
+    (pad "1" thru_hole roundrect (at 0 0 180) (size 1.7 2.032) (drill 0.95) (layers *.Cu *.Mask) (roundrect_rratio 0.1470588235)
       (net 33 "Left In") (pinfunction "1") (pintype "passive"))
     (pad "2" thru_hole oval (at 2.5 0 180) (size 1.7 2.032) (drill 0.95) (layers *.Cu *.Mask)
