File: KiCad/TDA2005Amplifier/TDA2005Amplifier.kicad_sch (KiCad schematic)
At the start: 30 parts, among them J1 Audio In, U1 Vol R, U2 Vol L, U3 TDA2005, U4 Speakers, U5 Power In

Commit message: PCBs
Connections:
- net OpOutR: now reaches C11.2, C6.2, C9.1, R4.1, U3.10
- net Op11: now reaches C6.1, U3.11 (BOOT)
- net Op7: now reaches C4.1, U3.7 (BOOT)
- net OpOutL: now reaches C10.2, C4.2, C8.1, R2.1, U3.8
Other:
- moved on the sheet: U4
Changed lines of the file:
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@@
 (kicad_sch (version 20211123) (generator eeschema)
   (paper "A4")
-  (junction (at 184.15 132.08) (diameter 0) (color 0 0 0 0)
-  )
   (junction (at 215.9 40.64) (diameter 0) (color 0 0 0 0)
   )
@@
   (junction (at 60.96 105.41) (diameter 0) (color 0 0 0 0)
   )
-  (junction (at 184.15 77.47) (diameter 0) (color 0 0 0 0)
-  )
   (junction (at 215.9 30.48) (diameter 0) (color 0 0 0 0)
   )
@@
   (junction (at 153.67 132.08) (diameter 0) (color 0 0 0 0)
   )
-  (junction (at 198.12 109.22) (diameter 0) (color 0 0 0 0)
+  (junction (at 245.11 148.59) (diameter 0) (color 0 0 0 0)
   )
   (junction (at 153.67 90.17) (diameter 0) (color 0 0 0 0)
@@
   (junction (at 153.67 144.78) (diameter 0) (color 0 0 0 0)
   )
-  (wire (pts (xy 184.15 132.08) (xy 210.82 132.08))
+  (wire (pts (xy 177.8 132.08) (xy 210.82 132.08))
     (stroke (width 0) (type default) (color 0 0 0 0))
   )
@@
     (stroke (width 0) (type default) (color 0 0 0 0))
   )
-  (wire (pts (xy 184.15 77.47) (xy 210.82 77.47))
+  (wire (pts (xy 177.8 77.47) (xy 210.82 77.47))
     (stroke (width 0) (type default) (color 0 0 0 0))
   )
@@
     (stroke (width 0) (type default) (color 0 0 0 0))
   )
-  (wire (pts (xy 177.8 132.08) (xy 184.15 132.08))
+  (wire (pts (xy 241.3 146.05) (xy 247.65 146.05))
     (stroke (width 0) (type default) (color 0 0 0 0))
   )
@@
     (stroke (width 0) (type default) (color 0 0 0 0))
   )
-  (wire (pts (xy 198.12 104.14) (xy 198.12 109.22))
+  (wire (pts (xy 245.11 143.51) (xy 245.11 148.59))
     (stroke (width 0) (type default) (color 0 0 0 0))
   )
@@
     (stroke (width 0) (type default) (color 0 0 0 0))
   )
-  (wire (pts (xy 184.15 106.68) (xy 200.66 106.68))
-    (stroke (width 0) (type default) (color 0 0 0 0))
-  )
-  (wire (pts (xy 200.66 104.14) (xy 198.12 104.14))
+  (wire (pts (xy 241.3 140.97) (xy 247.65 140.97))
+    (stroke (width 0) (type default) (color 0 0 0 0))
+  )
+  (wire (pts (xy 247.65 143.51) (xy 245.11 143.51))
     (stroke (width 0) (type default) (color 0 0 0 0))
   )
@@
     (stroke (width 0) (type default) (color 0 0 0 0))
   )
-  (wire (pts (xy 200.66 101.6) (xy 184.15 101.6))
-    (stroke (width 0) (type default) (color 0 0 0 0))
-  )
   (wire (pts (xy 66.04 74.93) (xy 66.04 83.82))
     (stroke (width 0) (type default) (color 0 0 0 0))
@@
     (stroke (width 0) (type default) (color 0 0 0 0))
   )
-  (wire (pts (xy 198.12 109.22) (xy 200.66 109.22))
+  (wire (pts (xy 245.11 148.59) (xy 247.65 148.59))
     (stroke (width 0) (type default) (color 0 0 0 0))
   )
@@
     (stroke (width 0) (type default) (color 0 0 0 0))
   )
-  (wire (pts (xy 177.8 77.47) (xy 184.15 77.47))
-    (stroke (width 0) (type default) (color 0 0 0 0))
-  )
   (wire (pts (xy 215.9 40.64) (xy 220.98 40.64))
     (stroke (width 0) (type default) (color 0 0 0 0))
@@
     (stroke (width 0) (type default) (color 0 0 0 0))
   )
-  (wire (pts (xy 184.15 106.68) (xy 184.15 132.08))
-    (stroke (width 0) (type default) (color 0 0 0 0))
-  )
   (wire (pts (xy 215.9 30.48) (xy 213.36 30.48))
     (stroke (width 0) (type default) (color 0 0 0 0))
   )
-  (wire (pts (xy 198.12 109.22) (xy 198.12 111.76))
+  (wire (pts (xy 245.11 148.59) (xy 245.11 151.13))
     (stroke (width 0) (type default) (color 0 0 0 0))
   )
@@
     (stroke (width 0) (type default) (color 0 0 0 0))
   )
-  (wire (pts (xy 184.15 101.6) (xy 184.15 77.47))
-    (stroke (width 0) (type default) (color 0 0 0 0))
-  )
   (wire (pts (xy 153.67 132.08) (xy 165.1 132.08))
     (stroke (width 0) (type default) (color 0 0 0 0))
@@
   (wire (pts (xy 138.43 57.15) (xy 149.86 57.15))
     (stroke (width 0) (type default) (color 0 0 0 0))
+  )
+  (label "Op11" (at 143.51 69.85 0)
+    (effects (font (size 1.27 1.27)) (justify left bottom))
+  )
+  (label "OpOutL" (at 156.21 132.08 0)
+    (effects (font (size 1.27 1.27)) (justify left bottom))
+  )
+  (label "Op7" (at 143.51 124.46 0)
+    (effects (font (size 1.27 1.27)) (justify left bottom))
+  )
+  (label "OpOutR" (at 156.21 77.47 0)
+    (effects (font (size 1.27 1.27)) (justify left bottom))
   )
   (global_label "Lin" (shape input) (at 43.18 100.33 180) (fields_autoplaced)
     (effects (font (size 1.27 1.27)) (justify right))
     (property "Intersheet References" "${INTERSHEET_REFS}" (id 0) (at 0 0 0)
+      (effects (font (size 1.27 1.27)) hide)
+    )
+  )
+  (global_label "Lout" (shape input) (at 241.3 146.05 180) (fields_autoplaced)
+    (effects (font (size 1.27 1.27)) (justify right))
+    (property "Intersheet References" "${INTERSHEET_REFS}" (id 0) (at 452.12 278.13 0)
+      (effects (font (size 1.27 1.27)) hide)
+    )
+  )
+  (global_label "Rout" (shape input) (at 241.3 140.97 180) (fields_autoplaced)
+    (effects (font (size 1.27 1.27)) (justify right))
+    (property "Intersheet References" "${INTERSHEET_REFS}" (id 0) (at 452.12 218.44 0)
       (effects (font (size 1.27 1.27)) hide)
     )
@@
     (pin "1")
   )
-  (symbol (lib_id "My_Parts:4-pole_RL-output_screw_terminal") (at 200.66 101.6 0) (unit 1)
-    (in_bom yes) (on_board yes)
-    (property "Reference" "U4" (id 0) (at 212.8012 104.1146 0)
-      (effects (font (size 1.27 1.27)) (justify left))
-    )
-    (property "Value" "Speakers" (id 1) (at 212.8012 106.426 0)
-      (effects (font (size 1.27 1.27)) (justify left))
-    )
-    (property "Footprint" "My_Parts:4-pole_screw_terminal_RL_output" (id 2) (at 205.105 98.425 0)
-      (effects (font (size 1.27 1.27)) hide)
-    )
-    (property "Datasheet" "" (id 3) (at 205.105 98.425 0)
+  (symbol (lib_id "My_Parts:4-pole_RL-output_screw_terminal") (at 247.65 140.97 0) (unit 1)
+    (in_bom yes) (on_board yes)
+    (property "Reference" "U4" (id 0) (at 259.7912 143.4846 0)
+      (effects (font (size 1.27 1.27)) (justify left))
+    )
+    (property "Value" "Speakers" (id 1) (at 259.7912 145.796 0)
+      (effects (font (size 1.27 1.27)) (justify left))
+    )
+    (property "Footprint" "My_Parts:4-pole_screw_terminal_RL_output" (id 2) (at 252.095 137.795 0)
+      (effects (font (size 1.27 1.27)) hide)
+    )
+    (property "Datasheet" "" (id 3) (at 252.095 137.795 0)
       (effects (font (size 1.27 1.27)) hide)
     )
@@
     (pin "4")
   )
-  (symbol (lib_id "power:GND") (at 198.12 111.76 0) (unit 1)
-    (in_bom yes) (on_board yes)
-    (property "Reference" "#PWR0109" (id 0) (at 198.12 118.11 0)
-      (effects (font (size 1.27 1.27)) hide)
-    )
-    (property "Value" "GND" (id 1) (at 198.247 116.1542 0))
-    (property "Footprint" "" (id 2) (at 198.12 111.76 0)
-      (effects (font (size 1.27 1.27)) hide)
-    )
-    (property "Datasheet" "" (id 3) (at 198.12 111.76 0)
-      (effects (font (size 1.27 1.27)) hide)
-    )
+  (symbol (lib_id "power:GND") (at 245.11 151.13 0) (unit 1)
+    (in_bom yes) (on_board yes)
+    (property "Reference" "#PWR0109" (id 0) (at 245.11 157.48 0)
+      (effects (font (size 1.27 1.27)) hide)
+    )
+    (property "Value" "GND" (id 1) (at 245.237 155.5242 0))
+    (property "Footprint" "" (id 2) (at 245.11 151.13 0)
+      (effects (font (size 1.27 1.27)) hide)
+    )
+    (property "Datasheet" "" (id 3) (at 245.11 151.13 0)
+      (effects (font (size 1.27 1.27)) hide)
+    )
