File: KiCad/ardAudioCenter/ardAudioCenter.kicad_sch (KiCad schematic)
At the start: 29 parts, among them J1 2-pin_power_input_header, J2 AudioPlug3, J3 4-pin_I2C_LCD_header, U1 2-pole_power_in_screw_terminal, U10 CD4052B, U11 MCP41010, U12 4-pole_RL-input_screw_terminal, U13 4-pole_RL-input_screw_terminal, U14 4-pole_RL-input_screw_terminal, U15 TEA5767_FM_Radio_Module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

Commit message: kicad
Parts:
- R3: footprint (none) -> My_Misc:R_Axial_DIN0207_L6.3mm_D2.5mm_P10.16mm_Horizontal_larger_pads
- U16, U9: footprint My_Headers:3-pin_potentiometer_header_larger_pads -> My_Headers:3-pin JST Potentiometer
Changed lines of the file:
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@@
       (effects (font (size 1.27 1.27)) (justify left))
     )
-    (property "Footprint" "My_Headers:3-pin_potentiometer_header_larger_pads" (id 2) (at 248.285 133.35 0)
+    (property "Footprint" "My_Headers:3-pin JST Potentiometer" (id 2) (at 248.285 133.35 0)
       (effects (font (size 1.27 1.27)) hide)
     )
@@
       (effects (font (size 1.27 1.27)) (justify left))
     )
-    (property "Footprint" "My_Headers:3-pin_potentiometer_header_larger_pads" (id 2) (at 193.675 133.35 0)
+    (property "Footprint" "My_Headers:3-pin JST Potentiometer" (id 2) (at 193.675 133.35 0)
       (effects (font (size 1.27 1.27)) hide)
     )
@@
       (effects (font (size 1.27 1.27)) (justify right))
     )
-    (property "Footprint" "" (id 2) (at 107.188 133.35 90)
+    (property "Footprint" "My_Misc:R_Axial_DIN0207_L6.3mm_D2.5mm_P10.16mm_Horizontal_larger_pads" (id 2) (at 107.188 133.35 90)
       (effects (font (size 1.27 1.27)) hide)
     )
@@
     )
     (path "/00000000-0000-0000-0000-00005eea47b7"
-      (reference "R3") (unit 1) (value "330R") (footprint "")
+      (reference "R3") (unit 1) (value "330R") (footprint "My_Misc:R_Axial_DIN0207_L6.3mm_D2.5mm_P10.16mm_Horizontal_larger_pads")
     )
     (path "/00000000-0000-0000-0000-00005ee57baf"
@@
     )
     (path "/00000000-0000-0000-0000-00005ee9ceae"
-      (reference "U9") (unit 1) (value "VolL") (footprint "My_Headers:3-pin_potentiometer_header_larger_pads")
+      (reference "U9") (unit 1) (value "VolL") (footprint "My_Headers:3-pin JST Potentiometer")
     )
     (path "/00000000-0000-0000-0000-00005ecc0ed1"
@@
     )
     (path "/00000000-0000-0000-0000-00005ee9c6fe"
-      (reference "U16") (unit 1) (value "VolR") (footprint "My_Headers:3-pin_potentiometer_header_larger_pads")
-    )
-  )
+      (reference "U16") (unit 1) (value "VolR") (footprint "My_Headers:3-pin JST Potentiometer")
+    )
+  )

Commit message: PCBs
Parts:
- removed C1: 0.33u, My_Misc:C_Disc_D7.5mm_W2.5mm_P5.00mm_larger, symbol Device:C
- removed C4: 0.1u, My_Misc:C_Disc_D7.5mm_W2.5mm_P5.00mm_larger, symbol Device:C
- removed J1: 2-pin_power_input_header, My_Headers:2-pin_power_input_header, symbol My_Headers:2-pin_power_input_header
- removed U12, U14: 4-pole_RL-input_screw_terminal, symbol My_Parts:4-pole_RL-input_screw_terminal
- removed U13: 4-pole_RL-input_screw_terminal, My_Parts:4-pole_screw_terminal_RL_input, symbol My_Parts:4-pole_RL-input_screw_terminal
- removed U3: L7805, My_Misc:TO-220-3_Vertical_larger, symbol Regulator_Linear:L7805
- removed U7: 4-pole_RL-output_screw_terminal, My_Parts:4-pole_screw_terminal_RL_output, symbol My_Parts:4-pole_RL-output_screw_terminal
- added C1: 10u, My_Misc:CP_Radial_D5.0mm_P2.00mm_larger, symbol Device:C_Polarized
- added C4: 22u, My_Misc:CP_Radial_D5.0mm_P2.00mm_larger, symbol Device:C_Polarized
- added H1, H2, H3, H4: MountingHole, MountingHole:MountingHole_3.5mm, symbol Mechanical:MountingHole
- added J2: Audio out, My_Headers:3-pin JST Audio, symbol My_Headers:3-pin_Audio
- added J4: FM In, My_Headers:3-pin JST Audio, symbol My_Headers:3-pin_Audio
- added J5: Line In, My_Headers:3-pin JST Audio, symbol My_Headers:3-pin_Audio
- added U3: AMS1117-5.0, Package_TO_SOT_SMD:SOT-223-3_TabPin2, symbol Regulator_Linear:AMS1117-5.0
- J1: renamed from J2; value AudioPlug3 -> FM Audio Plug
- J3: value 4-pin_I2C_LCD_header -> LCD; footprint My_Headers:4-pin_I2C_LCD_header_larger -> My_Headers:4-pin JST LCD
- U1: value 2-pole_power_in_screw_terminal -> Power In
- U10: renamed from U11; footprint My_Misc:DIP-8_W7.62mm_large -> My_Misc:DIP-8_W7.62mm_Socket_w_dip_packet_LongPads
- U12: renamed from U15; value TEA5767_FM_Radio_Module -> FM Radio TEA5767; footprint My_Headers:4-pin_TEA5767_radio_module_header_large -> My_Headers:4-pin JST TEA5767 FM Radio
- U2: value KY-040_Rotary_Encoder -> Rotary encoder 2; footprint My_Headers:5-pin_KY-040_rotary_encoder_header_larger -> My_Headers:5-pin JST Rotary Encoder
- U4: footprint (none) -> My_Headers:8-pin JST DFPlayer Mini
- U5: value KY-040_Rotary_Encoder -> Rotary encoder 1; footprint My_Headers:5-pin_KY-040_rotary_encoder_header_larger -> My_Headers:5-pin JST Rotary Encoder
- U6: footprint My_Headers:5-pin_JDY-62_bluetooth_module_header_large -> My_Headers:6-pin JST JDY-62 Bluetooth
- U7: renamed from U8; footprint My_Misc:DIP-8_W7.62mm_large -> My_Misc:DIP-8_W7.62mm_Socket_w_dip_packet_LongPads
- U9: renamed from U10; footprint My_Misc:DIP-16_W7.62mm_larger -> My_Misc:DIP-16_W7.62mm_LongPads w socket
- renumbered U16 to U11, U9 to U8
Connections:
- net +12V: now also C1.1, U3.3 (VI)
- net +5V: now also C4.1, U3.2 (VO)
- net FML+: no longer U9.1 (Y0)
- net FMR+: no longer U9.12 (X0)
- net GND: now also J3.2 (GND), C1.2, C4.2, J2.3 (-), J4.3 (-), J5.3 (-), U3.1 (GND); no longer J3.3 (GND)
- net Lout+: now also J2.2 (L+)
- net Rout+: now also J2.1 (R+)
- net SCL: now also J3.4 (SCL); no longer J3.7 (SCL)
- net SDA: now also J3.3 (SDA); no longer J3.5 (SDA)
- net LineL+: no longer names the net of U9.2 (Y2)
- net LineL+: now also J5.2 (L+)
- net LineR+: no longer names the net of U9.15 (X2)
- net LineR+: now also J5.1 (R+)
- new net: J4.2 (L+), U9.1 (Y0)
- new net: J4.1 (R+), U9.12 (X0)
Other:
- note removed: "This is to power the JDY-62 module"
- moved on the sheet: U12

Commit message: schematics
Parts:
- added Q1: BS170, My_Misc:TO-92_Inline_Wide_large, symbol Transistor_FET:BS170
- added R4: 220R, My_Misc:R_Axial_DIN0207_L6.3mm_D2.5mm_P10.16mm_Horizontal_larger_pads, symbol Device:R
Connections:
- net GND: now also Q1.3 (S); no longer U6.2 (GND)
- net BT-On: now reaches A1.15 (D12)
- net BT-On: now also R4.1
- new net: Q1.1 (D), U6.2 (GND)
- new net: Q1.2 (G), R4.2
Other:
- moved on the sheet: U6

Commit message: kicad
Other:
- title: (none) -> ardAudioCenter
Changed lines of the file:
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@@
 (kicad_sch (version 20211123) (generator eeschema)
   (paper "A4")
+  (title_block
+    (title "ardAudioCenter")
+    (date "2022-09-09")
+    (rev "0.4")
+  )
   (junction (at 158.75 146.05) (diameter 0) (color 0 0 0 0)
   )
