File: KiCad/ardAudioCenter-ATmega328/ATmega328.kicad_sch (KiCad schematic)
At the start: 7 parts, among them J1 FTDI, U2 ATmega328P-PU, Y1 16MHz

Commit message: kicad
Other:
- title: (none) -> ardAudioCenter-ATmega328
Changed lines of the file:
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@@
 (kicad_sch (version 20211123) (generator eeschema)
   (paper "A4")
+  (title_block
+    (title "ardAudioCenter-ATmega328")
+    (date "2022-09-09")
+    (rev "0.1")
+  )
   (junction (at 220.98 134.62) (diameter 0) (color 0 0 0 0)
   )
