File: KiCad/ardAudioCenter-ATmega328/ardAudioCenter-ATmega328.kicad_pcb (KiCad board)
At the start: 2 copper layers, 101 x 70.5 mm, 38 parts, among them J1 FTDI, J4 Audio out, J5 LCD, J6 FM In, J7 Line In, Q1 BS170, U10 VolL, U11 CD4052B, U12 MCP41010, U13 VolR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

Commit message: kicad
Other:
- board text added: "${TITLE}-${REVISION} Design: Jon Sagebrand github.com/jonsag"
- board text removed: "ardAudioCenter-Atmega328-0.1 Design: Jon Sagebrand github.com/jonsag"
Changed lines of the file:
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@@
   )
   (paper "A4")
+  (title_block
+    (title "ardAudioCenter-ATmega328")
+    (date "2022-09-09")
+    (rev "0.1")
+  )
   (layers
     (0 "F.Cu" signal)
@@
   (gr_arc (start 118.11 146.05) (mid 114.96691 144.74809) (end 113.665 141.605) (layer "Edge.Cuts") (width 0.1))
   (gr_arc (start 113.665 80.01) (mid 114.96691 76.86691) (end 118.11 75.565) (layer "Edge.Cuts") (width 0.1))
-  (gr_text "ardAudioCenter-Atmega328-0.1\nDesign: Jon Sagebrand\ngithub.com/jonsag" (at 210.185 127 90) (layer "F.SilkS")
+  (gr_text "${TITLE}-${REVISION}\nDesign: Jon Sagebrand\ngithub.com/jonsag" (at 210.185 127 90) (layer "F.SilkS")
     (effects (font (size 1 1) (thickness 0.15)) (justify left))
   )
