File: KiCad/ardAudioCenter-ATmega328/ardAudioCenter-ATmega328.kicad_sch (KiCad schematic)
At the start: 32 parts, among them J3 FM Audio Plug, J4 Audio out, J5 LCD, J6 FM In, J7 Line In, Q1 BS170, U10 VolL, U11 CD4052B, U12 MCP41010, U13 VolR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

Commit message: kicad
Other:
- note added: "ATmega328P"
- title: (none) -> ardAudioCenter-ATmega328
Changed lines of the file:
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@@
 (kicad_sch (version 20211123) (generator eeschema)
   (paper "A4")
+  (title_block
+    (title "ardAudioCenter-ATmega328")
+    (date "2022-09-09")
+    (rev "0.1")
+  )
   (junction (at 156.21 142.24) (diameter 0) (color 0 0 0 0)
   )
@@
     (stroke (width 0) (type default) (color 0 0 0 0))
   )
+  (polyline (pts (xy 121.92 85.09) (xy 149.86 85.09))
+    (stroke (width 0) (type default) (color 0 0 0 0))
+  )
   (wire (pts (xy 186.69 107.95) (xy 186.69 96.52))
     (stroke (width 0) (type default) (color 0 0 0 0))
@@
     (stroke (width 0) (type default) (color 0 0 0 0))
   )
+  (polyline (pts (xy 121.92 85.09) (xy 121.92 118.11))
+    (stroke (width 0) (type default) (color 0 0 0 0))
+  )
   (wire (pts (xy 86.36 76.2) (xy 86.36 66.04))
     (stroke (width 0) (type default) (color 0 0 0 0))
@@
     (stroke (width 0) (type default) (color 0 0 0 0))
   )
+  (polyline (pts (xy 149.86 118.11) (xy 149.86 85.09))
+    (stroke (width 0) (type default) (color 0 0 0 0))
+  )
   (wire (pts (xy 64.77 120.65) (xy 92.71 120.65))
     (stroke (width 0) (type default) (color 0 0 0 0))
@@
     (stroke (width 0) (type default) (color 0 0 0 0))
   )
+  (polyline (pts (xy 121.92 118.11) (xy 149.86 118.11))
+    (stroke (width 0) (type default) (color 0 0 0 0))
+  )
   (wire (pts (xy 78.74 78.74) (xy 86.36 78.74))
     (stroke (width 0) (type default) (color 0 0 0 0))
@@
   )
   (text "This connects to Audio out\non TEA5767 module" (at 86.36 34.29 0)
+    (effects (font (size 1.27 1.27)) (justify left bottom))
+  )
+  (text "ATmega328P" (at 135.89 88.9 0)
     (effects (font (size 1.27 1.27)) (justify left bottom))
   )
@@
   (symbol (lib_id "My_Parts:JDY-62_Bluetooth_Module") (at 135.89 161.29 0) (unit 1)
     (in_bom yes) (on_board yes)
-    (property "Reference" "U8" (id 0) (at 148.5392 186.6646 0)
-      (effects (font (size 1.27 1.27)) (justify left))
-    )
-    (property "Value" "JDY-62_Bluetooth_Module" (id 1) (at 148.5392 188.976 0)
+    (property "Reference" "U8" (id 0) (at 146.05 166.37 0)
+      (effects (font (size 1.27 1.27)) (justify left))
+    )
+    (property "Value" "JDY-62_Bluetooth_Module" (id 1) (at 146.05 168.6814 0)
       (effects (font (size 1.27 1.27)) (justify left))
     )
@@
     (pin "2")
   )
-  (sheet (at 146.05 186.69) (size 12.7 3.81) (fields_autoplaced)
+  (sheet (at 147.32 186.69) (size 12.7 3.81) (fields_autoplaced)
     (stroke (width 0.1524) (type solid) (color 0 0 0 0))
     (fill (color 0 0 0 0.0000))
-    (property "Sheet name" "ATmega328" (id 0) (at 146.05 185.9784 0)
+    (property "Sheet name" "ATmega328" (id 0) (at 147.32 185.9784 0)
       (effects (font (size 1.27 1.27)) (justify left bottom))
     )
-    (property "Sheet file" "ATmega328.kicad_sch" (id 1) (at 146.05 191.0846 0)
+    (property "Sheet file" "ATmega328.kicad_sch" (id 1) (at 147.32 191.0846 0)
       (effects (font (size 1.27 1.27)) (justify left top))
     )
